Commit message: minor update on livox model

File: urdf/mid360.xacro (robot description, xacro)
@@ -3,5 +3,5 @@
   <xacro:property name="M_PI" value="3.1415926"/>
   <xacro:property name="laser_min_range" value="0.1"/>
-  <xacro:property name="laser_max_range" value="200.0"/>
+  <xacro:property name="laser_max_range" value="20.0"/>
   <xacro:property name="samples" value="40000"/>
   <xacro:property name="resolution" value="0.002"/>
@@ -20,12 +20,12 @@
   </xacro:macro>
   <xacro:macro name="mid360" params="name:='' parent:= 'base_link' topic:='mid360' *origin ">
-<link name="${name}">
-<xacro:box_inertia m="${length}" w="${width}" d="${length}" h="${height}"/>
-  <visual>
-        <geometry>
-            <box size="${length} ${width} ${height}"/>
-        </geometry>
-  </visual>
-</link>
+  <link name="${name}">
+  <xacro:box_inertia m="${length}" w="${width}" d="${length}" h="${height}"/>
+    <visual>
+          <geometry>
+              <box size="${length} ${width} ${height}"/>
+          </geometry>
+    </visual>
+  </link>
     <joint name="${name}_joint" type="fixed">
       <parent link="${parent}"/>
@@ -40,30 +40,30 @@
         <!-- This ray plgin is only for visualization. -->
         <plugin name="${name}_plugin" filename="libros2_livox.so">
-			<ray>
-			  <scan>
-				<horizontal>
-				<samples>100</samples>
-				<resolution>1</resolution>
-				<min_angle>${0}</min_angle>
-				<max_angle>${2*M_PI}</max_angle>
-				</horizontal>
-				<vertical>
-				<samples>360</samples>
-				<resolution>1</resolution>
-				<min_angle>${-7.22/180*M_PI}</min_angle>
-				<max_angle>${55.22/180*M_PI}</max_angle>
-				</vertical>
-			  </scan>
-			  <range>
-				<min>${laser_min_range}</min>
-				<max>${laser_max_range}</max>
-				<resolution>${resolution}</resolution>
-			  </range>
-			  <noise>
-				<type>gaussian</type>
-				<mean>${noise_mean}</mean>
-				<stddev>${noise_stddev}</stddev>
-			  </noise>
-			</ray>
+        <ray>
+          <scan>
+          <horizontal>
+          <samples>100</samples>
+          <resolution>1</resolution>
+          <min_angle>${0}</min_angle>
+          <max_angle>${2*M_PI}</max_angle>
+          </horizontal>
+          <vertical>
+          <samples>360</samples>
+          <resolution>1</resolution>
+          <min_angle>${-7.22/180*M_PI}</min_angle>
+          <max_angle>${55.22/180*M_PI}</max_angle>
+          </vertical>
+          </scan>
+          <range>
+          <min>${laser_min_range}</min>
+          <max>${laser_max_range}</max>
+          <resolution>${resolution}</resolution>
+          </range>
+          <noise>
+          <type>gaussian</type>
+          <mean>${noise_mean}</mean>
+          <stddev>${noise_stddev}</stddev>
+          </noise>
+        </ray>
           <visualize>false</visualize>
 		  <samples>${samples}</samples>
@@ -73,4 +73,5 @@
         </plugin>
       </sensor>
+      <gravity>0</gravity>
     </gazebo>
   </xacro:macro>

Commit message: remove livox visual

File: urdf/mid360.xacro (robot description, xacro)
@@ -2,6 +2,6 @@
 <robot xmlns:xacro="http://ros.org/wiki/xacro">
   <xacro:property name="M_PI" value="3.1415926"/>
-  <xacro:property name="laser_min_range" value="0.1"/>
-  <xacro:property name="laser_max_range" value="20.0"/>
+  <xacro:property name="laser_min_range" value="0.2"/>
+  <xacro:property name="laser_max_range" value="10.0"/>
   <xacro:property name="samples" value="40000"/>
   <xacro:property name="resolution" value="0.002"/>
@@ -22,9 +22,10 @@
   <link name="${name}">
   <xacro:box_inertia m="${length}" w="${width}" d="${length}" h="${height}"/>
-    <visual>
+    <!-- Removed the visual element for the box -->
+    <!-- <visual>
           <geometry>
               <box size="${length} ${width} ${height}"/>
           </geometry>
-    </visual>
+    </visual> -->
   </link>
     <joint name="${name}_joint" type="fixed">
@@ -36,7 +37,7 @@
       <sensor type="ray" name="${name}">
         <pose>0 0 0 0 0 0</pose>
-        <visualize>true</visualize>
-        <update_rate>10</update_rate>
-        <!-- This ray plgin is only for visualization. -->
+        <visualize>true</visualize>  <!-- Ensure no sensor visualization -->
+        <update_rate>30</update_rate>
+        <!-- This ray plugin is for sensor data -->
         <plugin name="${name}_plugin" filename="libros2_livox.so">
         <ray>

Commit message: sim ready code

File: urdf/mid360.xacro (robot description, xacro)
@@ -2,8 +2,8 @@
 <robot xmlns:xacro="http://ros.org/wiki/xacro">
   <xacro:property name="M_PI" value="3.1415926"/>
-  <xacro:property name="laser_min_range" value="0.2"/>
+  <xacro:property name="laser_min_range" value="0.01"/>
   <xacro:property name="laser_max_range" value="10.0"/>
-  <xacro:property name="samples" value="40000"/>
-  <xacro:property name="resolution" value="0.002"/>
+  <xacro:property name="samples" value="5000"/>
+  <xacro:property name="resolution" value="0.1"/>
   <xacro:property name="noise_mean" value="0.0"/>
   <xacro:property name="noise_stddev" value="0.01"/>
@@ -19,5 +19,5 @@
     </inertial>
   </xacro:macro>
-  <xacro:macro name="mid360" params="name:='' parent:= 'base_link' topic:='mid360' *origin ">
+  <xacro:macro name="mid360" params="name:='' namespace:='NX01' parent:= 'base_link' topic:='mid360' *origin ">
   <link name="${name}">
   <xacro:box_inertia m="${length}" w="${width}" d="${length}" h="${height}"/>
@@ -71,5 +71,5 @@
 		  <downsample>1</downsample>
 		  <csv_file_name>$(find ros2_livox_simulation)/scan_mode/mid360.csv</csv_file_name>
-		  <topic>${topic}</topic>
+		  <topic>${namespace}/${topic}</topic>
         </plugin>
       </sensor>

Commit message: multiagent

File: urdf/mid360.xacro (robot description, xacro)
@@ -19,5 +19,5 @@
     </inertial>
   </xacro:macro>
-  <xacro:macro name="mid360" params="name:='' namespace:='NX01' parent:= 'base_link' topic:='mid360' *origin ">
+  <xacro:macro name="mid360" params="name:='' namespace:='quadrotor' parent:= 'base_link' topic:='mid360' *origin ">
   <link name="${name}">
   <xacro:box_inertia m="${length}" w="${width}" d="${length}" h="${height}"/>
@@ -42,35 +42,36 @@
         <!-- This ray plugin is for sensor data -->
         <plugin name="${name}_plugin" filename="libros2_livox.so">
-        <ray>
-          <scan>
-          <horizontal>
-          <samples>100</samples>
-          <resolution>1</resolution>
-          <min_angle>${0}</min_angle>
-          <max_angle>${2*M_PI}</max_angle>
-          </horizontal>
-          <vertical>
-          <samples>360</samples>
-          <resolution>1</resolution>
-          <min_angle>${-7.22/180*M_PI}</min_angle>
-          <max_angle>${55.22/180*M_PI}</max_angle>
-          </vertical>
-          </scan>
-          <range>
-          <min>${laser_min_range}</min>
-          <max>${laser_max_range}</max>
-          <resolution>${resolution}</resolution>
-          </range>
-          <noise>
-          <type>gaussian</type>
-          <mean>${noise_mean}</mean>
-          <stddev>${noise_stddev}</stddev>
-          </noise>
-        </ray>
+          <ray>
+            <scan>
+            <horizontal>
+            <samples>100</samples>
+            <resolution>1</resolution>
+            <min_angle>${0}</min_angle>
+            <max_angle>${2*M_PI}</max_angle>
+            </horizontal>
+            <vertical>
+            <samples>360</samples>
+            <resolution>1</resolution>
+            <min_angle>${-7.22/180*M_PI}</min_angle>
+            <max_angle>${55.22/180*M_PI}</max_angle>
+            </vertical>
+            </scan>
+            <range>
+            <min>${laser_min_range}</min>
+            <max>${laser_max_range}</max>
+            <resolution>${resolution}</resolution>
+            </range>
+            <noise>
+            <type>gaussian</type>
+            <mean>${noise_mean}</mean>
+            <stddev>${noise_stddev}</stddev>
+            </noise>
+          </ray>
           <visualize>false</visualize>
-		  <samples>${samples}</samples>
-		  <downsample>1</downsample>
-		  <csv_file_name>$(find ros2_livox_simulation)/scan_mode/mid360.csv</csv_file_name>
-		  <topic>${namespace}/${topic}</topic>
+		      <samples>${samples}</samples>
+		      <downsample>1</downsample>
+		      <csv_file_name>$(find ros2_livox_simulation)/scan_mode/mid360.csv</csv_file_name>
+		      <topic>${topic}</topic>
+          <namespace>${namespace}</namespace>
         </plugin>
       </sensor>

Commit message: imu added for dlio

File: urdf/mid360.xacro (robot description, xacro)
@@ -4,5 +4,5 @@
   <xacro:property name="laser_min_range" value="0.01"/>
   <xacro:property name="laser_max_range" value="10.0"/>
-  <xacro:property name="samples" value="5000"/>
+  <xacro:property name="samples" value="20000"/>
   <xacro:property name="resolution" value="0.1"/>
   <xacro:property name="noise_mean" value="0.0"/>
@@ -14,19 +14,20 @@
   <xacro:macro name="box_inertia" params="m w h d">
     <inertial>
-      <origin xyz="0 0 0" rpy="${pi/2} 0 ${pi/2}"/>
+      <origin xyz="0 0 0" rpy="0 0 0"/>
       <mass value="${m}"/>
       <inertia ixx="${(m/12) * (h*h + d*d)}" ixy="0.0" ixz="0.0" iyy="${(m/12) * (w*w + d*d)}" iyz="0.0" izz="${(m/12) * (w*w + h*h)}"/>
     </inertial>
   </xacro:macro>
-  <xacro:macro name="mid360" params="name:='' namespace:='quadrotor' parent:= 'base_link' topic:='mid360' *origin ">
-  <link name="${name}">
-  <xacro:box_inertia m="${length}" w="${width}" d="${length}" h="${height}"/>
-    <!-- Removed the visual element for the box -->
-    <!-- <visual>
-          <geometry>
-              <box size="${length} ${width} ${height}"/>
-          </geometry>
-    </visual> -->
-  </link>
+  <xacro:macro name="mid360" params=" name:=''
+                                      namespace:='quadrotor'
+                                      parent:='base_link'
+                                      topic:='mid360'
+                                      *origin
+                                      accel_fps:=250
+                                      gyro_fps:=500
+                                      ">
+    <link name="${name}">
+      <xacro:box_inertia m="${length}" w="${width}" d="${length}" h="${height}"/>
+    </link>
     <joint name="${name}_joint" type="fixed">
       <parent link="${parent}"/>
@@ -39,5 +40,5 @@
         <always_on>true</always_on>
         <visualize>false</visualize>  <!-- Ensure no sensor visualization -->
-        <update_rate>30</update_rate>
+        <update_rate>200</update_rate>
         <!-- This ray plugin is for sensor data -->
         <plugin name="${name}_plugin" filename="libros2_livox.so">
@@ -69,11 +70,58 @@
           </ray>
           <visualize>false</visualize>
-		      <samples>${samples}</samples>
-		      <downsample>1</downsample>
-		      <csv_file_name>$(find ros2_livox_simulation)/scan_mode/mid360.csv</csv_file_name>
-		      <topic>${topic}</topic>
+          <samples>${samples}</samples>
+          <downsample>1</downsample>
+          <csv_file_name>$(find ros2_livox_simulation)/scan_mode/mid360.csv</csv_file_name>
+          <topic>${topic}</topic>
           <namespace>${namespace}</namespace>
         </plugin>
       </sensor>
+      <!-- IMU -->
+      <sensor name="${name}/imu" type="imu">
+        <always_on>true</always_on>
+        <update_rate>${gyro_fps}</update_rate>
+        <topic>${name}/imu/sample</topic>
+        <plugin name="${name}_imu" filename="libimu_plugin.so">
+          <topicName>${name}/imu/sample</topicName>
+          <bodyName>${name}_link</bodyName>
+          <updateRateHZ>${gyro_fps}</updateRateHZ>
+          <gaussianNoise>0.0</gaussianNoise>
+          <xyzOffset>0 0 0</xyzOffset>
+          <rpyOffset>0 0 0</rpyOffset>
+        </plugin>
+      </sensor>
+      <!-- Accel -->
+      <!-- <sensor name="${name}accel" type="imu">
+        <always_on>true</always_on>
+        <update_rate>${accel_fps}</update_rate>
+        <topic>${name}/accel/sample</topic>
+        <plugin name="${topics_ns}_accel_plugin" filename="librealsense_gazebo_accel_sensor.so">
+          <topicName>${name}/accel/sample</topicName>
+          <bodyName>${name}_link</bodyName>
+          <updateRateHZ>${accel_fps}</updateRateHZ>
+          <gaussianNoise>0.1</gaussianNoise>
+          <xyzOffset>0 0 0</xyzOffset>
+          <rpyOffset>0 0 0</rpyOffset>
+          <frameName>${parent}</frameName>
+          <initialOrientationAsReference>false</initialOrientationAsReference>
+        </plugin>
+        <pose>0 0 0 0 0 0</pose>
+      </sensor> -->
+      <!-- Gyro -->
+      <!-- <sensor name="${name}gyro" type="imu">
+        <always_on>true</always_on>
+        <update_rate>${gyro_fps}</update_rate>
+        <topic>${name}/gyro/sample</topic>
+        <plugin name="${topics_ns}_gyro_plugin" filename="librealsense_gazebo_gyro_sensor.so">
+          <topicName>${name}/gyro/sample</topicName>
+          <bodyName>${name}_link</bodyName>
+          <updateRateHZ>${gyro_fps}</updateRateHZ>
+          <gaussianNoise>0.1</gaussianNoise>
+          <xyzOffset>0 0 0</xyzOffset>
+          <rpyOffset>0 0 0</rpyOffset>
+          <frameName>${parent}</frameName>
+          <initialOrientationAsReference>false</initialOrientationAsReference>
+        </plugin>
+      </sensor> -->
       <gravity>0</gravity>
     </gazebo>

Commit message: sample number updated in mid360

File: urdf/mid360.xacro (robot description, xacro)
@@ -4,5 +4,5 @@
   <xacro:property name="laser_min_range" value="0.01"/>
   <xacro:property name="laser_max_range" value="10.0"/>
-  <xacro:property name="samples" value="20000"/>
+  <xacro:property name="samples" value="5000"/>
   <xacro:property name="resolution" value="0.1"/>
   <xacro:property name="noise_mean" value="0.0"/>

Commit message: forest high speed flight

File: urdf/mid360.xacro (robot description, xacro)
@@ -5,5 +5,5 @@
   <xacro:property name="laser_max_range" value="10.0"/>
   <xacro:property name="samples" value="5000"/>
-  <xacro:property name="resolution" value="0.1"/>
+  <xacro:property name="resolution" value="0.05s"/>
   <xacro:property name="noise_mean" value="0.0"/>
   <xacro:property name="noise_stddev" value="0.01"/>

Commit message: single agent exploration in cave

File: urdf/mid360.xacro (robot description, xacro)
@@ -4,5 +4,5 @@
   <xacro:property name="laser_min_range" value="0.01"/>
   <xacro:property name="laser_max_range" value="10.0"/>
-  <xacro:property name="samples" value="5000"/>
+  <xacro:property name="samples" value="10000"/>
   <xacro:property name="resolution" value="0.05s"/>
   <xacro:property name="noise_mean" value="0.0"/>

Commit message: roi map sharing done

File: urdf/mid360.xacro (robot description, xacro)
@@ -2,8 +2,8 @@
 <robot xmlns:xacro="http://ros.org/wiki/xacro">
   <xacro:property name="M_PI" value="3.1415926"/>
-  <xacro:property name="laser_min_range" value="0.01"/>
+  <xacro:property name="laser_min_range" value="0.001"/>
   <xacro:property name="laser_max_range" value="10.0"/>
-  <xacro:property name="samples" value="10000"/>
-  <xacro:property name="resolution" value="0.05s"/>
+  <xacro:property name="samples" value="5000"/>
+  <xacro:property name="resolution" value="0.05"/>
   <xacro:property name="noise_mean" value="0.0"/>
   <xacro:property name="noise_stddev" value="0.01"/>
@@ -78,5 +78,5 @@
       </sensor>
       <!-- IMU -->
-      <sensor name="${name}/imu" type="imu">
+      <!-- <sensor name="${name}/imu" type="imu">
         <always_on>true</always_on>
         <update_rate>${gyro_fps}</update_rate>
@@ -90,5 +90,5 @@
           <rpyOffset>0 0 0</rpyOffset>
         </plugin>
-      </sensor>
+      </sensor> -->
       <!-- Accel -->
       <!-- <sensor name="${name}accel" type="imu">

Commit message: max range is given by laser_max_range in xacro

File: urdf/mid360.xacro (robot description, xacro)
@@ -3,5 +3,5 @@
   <xacro:property name="M_PI" value="3.1415926"/>
   <xacro:property name="laser_min_range" value="0.001"/>
-  <xacro:property name="laser_max_range" value="10.0"/>
+  <xacro:property name="laser_max_range" value="30.0"/>
   <xacro:property name="samples" value="5000"/>
   <xacro:property name="resolution" value="0.05"/>
@@ -45,21 +45,21 @@
           <ray>
             <scan>
-            <horizontal>
-            <samples>100</samples>
-            <resolution>1</resolution>
-            <min_angle>${0}</min_angle>
-            <max_angle>${2*M_PI}</max_angle>
-            </horizontal>
+              <horizontal>
+                <samples>100</samples>
+                <resolution>1</resolution>
+                <min_angle>${0}</min_angle>
+                <max_angle>${2*M_PI}</max_angle>
+              </horizontal>
             <vertical>
-            <samples>360</samples>
-            <resolution>1</resolution>
-            <min_angle>${-7.22/180*M_PI}</min_angle>
-            <max_angle>${55.22/180*M_PI}</max_angle>
+              <samples>360</samples>
+              <resolution>1</resolution>
+              <min_angle>${-7.22/180*M_PI}</min_angle>
+              <max_angle>${55.22/180*M_PI}</max_angle>
             </vertical>
             </scan>
             <range>
-            <min>${laser_min_range}</min>
-            <max>${laser_max_range}</max>
-            <resolution>${resolution}</resolution>
+              <min>${laser_min_range}</min>
+              <max>${laser_max_range}</max>
+              <resolution>${resolution}</resolution>
             </range>
             <noise>

Commit message: light weight simulation

File: urdf/mid360.xacro (robot description, xacro)
@@ -4,6 +4,6 @@
   <xacro:property name="laser_min_range" value="0.001"/>
   <xacro:property name="laser_max_range" value="30.0"/>
-  <xacro:property name="samples" value="5000"/>
-  <xacro:property name="resolution" value="0.05"/>
+  <xacro:property name="samples" value="100"/>
+  <xacro:property name="resolution" value="0.1"/>
   <xacro:property name="noise_mean" value="0.0"/>
   <xacro:property name="noise_stddev" value="0.01"/>
@@ -40,5 +40,5 @@
         <always_on>true</always_on>
         <visualize>false</visualize>  <!-- Ensure no sensor visualization -->
-        <update_rate>200</update_rate>
+        <update_rate>100</update_rate>
         <!-- This ray plugin is for sensor data -->
         <plugin name="${name}_plugin" filename="libros2_livox.so">

Commit message: sample 3000 (same as in acl-sim for benchmarking)

File: urdf/mid360.xacro (robot description, xacro)
@@ -4,8 +4,8 @@
   <xacro:property name="laser_min_range" value="0.001"/>
   <xacro:property name="laser_max_range" value="30.0"/>
-  <xacro:property name="samples" value="100"/>
+  <xacro:property name="samples" value="3000"/>
   <xacro:property name="resolution" value="0.1"/>
   <xacro:property name="noise_mean" value="0.0"/>
-  <xacro:property name="noise_stddev" value="0.01"/>
+  <xacro:property name="noise_stddev" value="0.0"/>
   <xacro:property name="mass" value="0.4" />
   <xacro:property name="length" value="0.1" />

Commit message: benchmark is done

File: urdf/mid360.xacro (robot description, xacro)
@@ -3,6 +3,6 @@
   <xacro:property name="M_PI" value="3.1415926"/>
   <xacro:property name="laser_min_range" value="0.001"/>
-  <xacro:property name="laser_max_range" value="30.0"/>
-  <xacro:property name="samples" value="3000"/>
+  <xacro:property name="laser_max_range" value="10.0"/>
+  <xacro:property name="samples" value="2000"/>
   <xacro:property name="resolution" value="0.1"/>
   <xacro:property name="noise_mean" value="0.0"/>

Commit message: working with dynus repo mighty

File: urdf/mid360.xacro (robot description, xacro)
@@ -3,5 +3,5 @@
   <xacro:property name="M_PI" value="3.1415926"/>
   <xacro:property name="laser_min_range" value="0.001"/>
-  <xacro:property name="laser_max_range" value="10.0"/>
+  <xacro:property name="laser_max_range" value="15.0"/>
   <xacro:property name="samples" value="2000"/>
   <xacro:property name="resolution" value="0.1"/>

Commit message: DYNUS static benchmark

File: urdf/mid360.xacro (robot description, xacro)
@@ -3,7 +3,7 @@
   <xacro:property name="M_PI" value="3.1415926"/>
   <xacro:property name="laser_min_range" value="0.001"/>
-  <xacro:property name="laser_max_range" value="15.0"/>
-  <xacro:property name="samples" value="2000"/>
-  <xacro:property name="resolution" value="0.1"/>
+  <xacro:property name="laser_max_range" value="12.0"/>
+  <xacro:property name="samples" value="1000"/>
+  <xacro:property name="resolution" value="0.15"/>
   <xacro:property name="noise_mean" value="0.0"/>
   <xacro:property name="noise_stddev" value="0.0"/>

Commit message: larger range for livox

File: urdf/mid360.xacro (robot description, xacro)
@@ -3,5 +3,5 @@
   <xacro:property name="M_PI" value="3.1415926"/>
   <xacro:property name="laser_min_range" value="0.001"/>
-  <xacro:property name="laser_max_range" value="12.0"/>
+  <xacro:property name="laser_max_range" value="20.0"/>
   <xacro:property name="samples" value="1000"/>
   <xacro:property name="resolution" value="0.15"/>

Commit message: working with sando

File: urdf/mid360.xacro (robot description, xacro)
@@ -4,5 +4,5 @@
   <xacro:property name="laser_min_range" value="0.001"/>
   <xacro:property name="laser_max_range" value="20.0"/>
-  <xacro:property name="samples" value="1000"/>
+  <xacro:property name="samples" value="2000"/>
   <xacro:property name="resolution" value="0.15"/>
   <xacro:property name="noise_mean" value="0.0"/>
@@ -40,5 +40,5 @@
         <always_on>true</always_on>
         <visualize>false</visualize>  <!-- Ensure no sensor visualization -->
-        <update_rate>100</update_rate>
+        <update_rate>1000</update_rate>
         <!-- This ray plugin is for sensor data -->
         <plugin name="${name}_plugin" filename="libros2_livox.so">
@@ -72,4 +72,6 @@
           <samples>${samples}</samples>
           <downsample>1</downsample>
+          <accumulate_scans>5</accumulate_scans>
+          <num_phases>5</num_phases>
           <csv_file_name>$(find ros2_livox_simulation)/scan_mode/mid360.csv</csv_file_name>
           <topic>${topic}</topic>
